File: Minotaur/Hardware/Minotaur.kicad_sch (KiCad schematic)
At the start: 31 parts, among them J1 CELL BALANCE, J2 SWD, J3 UART, Q14 BSS84, Q6 CSD17501Q5A, Q7 CSD17501Q5A

Commit message: Vulkan Minotaur : Updated Hardware Schematic
Parts:
- removed R19: TBD, symbol Device:R_Shunt
- removed R22: 1M, symbol Device:R_Small
- removed R23: 1k, symbol Device:R_Small
- added BT?: 0SP2, Battery:BatteryHolder_MPD_BH-18650-PC2, symbol Device:Battery_Cell
- added BT?: 3SP1, Battery:BatteryHolder_MPD_BH-18650-PC2, symbol Device:Battery_Cell
- added BT?: 1SP1, Battery:BatteryHolder_MPD_BH-18650-PC2, symbol Device:Battery_Cell
- added BT?: 1SP2, Battery:BatteryHolder_MPD_BH-18650-PC2, symbol Device:Battery_Cell
- added BT?: 0SP1, Battery:BatteryHolder_MPD_BH-18650-PC2, symbol Device:Battery_Cell
- added BT?: 2SP2, Battery:BatteryHolder_MPD_BH-18650-PC2, symbol Device:Battery_Cell
- added BT?: 4SP2, Battery:BatteryHolder_MPD_BH-18650-PC2, symbol Device:Battery_Cell
- added BT?: 4SP1, Battery:BatteryHolder_MPD_BH-18650-PC2, symbol Device:Battery_Cell
- added BT?: 2SP1, Battery:BatteryHolder_MPD_BH-18650-PC2, symbol Device:Battery_Cell
- added BT?: 3SP2, Battery:BatteryHolder_MPD_BH-18650-PC2, symbol Device:Battery_Cell
- added C104, C105: 100n, Capacitor_SMD:C_0603_1608Metric_Pad1.08x0.95mm_HandSolder, symbol Device:C_Small
- added R102, R103, R104: R_Small, Resistor_SMD:R_2512_6332Metric_Pad1.40x3.35mm_HandSolder, symbol Device:R_Small
- BT?: renamed from BT1; value Battery_Cell -> 0SP0; footprint (none) -> Battery:BatteryHolder_MPD_BH-18650-PC2
- BT?: renamed from BT3; value Battery_Cell -> 2SP0; footprint (none) -> Battery:BatteryHolder_MPD_BH-18650-PC2
- BT?: renamed from BT5; value Battery_Cell -> 4SP0; footprint (none) -> Battery:BatteryHolder_MPD_BH-18650-PC2
- BT?: renamed from BT2; value Battery_Cell -> 1SP0; footprint (none) -> Battery:BatteryHolder_MPD_BH-18650-PC2
- BT?: renamed from BT4; value Battery_Cell -> 3SP0; footprint (none) -> Battery:BatteryHolder_MPD_BH-18650-PC2
- C?: renamed from C12; footprint (none) -> Capacitor_SMD:C_0603_1608Metric_Pad1.08x0.95mm_HandSolder
- C?: renamed from C8; footprint (none) -> Capacitor_SMD:C_0603_1608Metric_Pad1.08x0.95mm_HandSolder
- C?: renamed from C7; footprint (none) -> Capacitor_SMD:C_0603_1608Metric_Pad1.08x0.95mm_HandSolder
- C?: renamed from C13; footprint (none) -> Capacitor_SMD:C_0603_1608Metric_Pad1.08x0.95mm_HandSolder
- C?: renamed from C9; footprint (none) -> Capacitor_SMD:C_0603_1608Metric_Pad1.08x0.95mm_HandSolder
- D?: renamed from D6; footprint (none) -> Diode_SMD:D_SOD-123
- D?: renamed from D9; value D_Small -> MURS360T3G; footprint (none) -> Diode_SMD:D_SMC_Handsoldering
- D?: renamed from D7; value D_Small -> MMSD914T1G; footprint (none) -> Diode_SMD:D_SOD-123
- D?: renamed from D6; value D_TVS -> SMCJ57A; footprint (none) -> Diode_SMD:D_SMC_Handsoldering
- NT?: renamed from NT1; footprint (none) -> NetTie:NetTie-2_SMD_Pad2.0mm
- NT?: renamed from NT2; footprint (none) -> NetTie:NetTie-2_SMD_Pad2.0mm
- R?: renamed from R20; footprint (none) -> Resistor_SMD:R_0603_1608Metric_Pad0.98x0.95mm_HandSolder
- R?: renamed from R21; footprint (none) -> Resistor_SMD:R_0603_1608Metric_Pad0.98x0.95mm_HandSolder
- R?: renamed from R18; footprint (none) -> Resistor_SMD:R_0603_1608Metric_Pad0.98x0.95mm_HandSolder
- R?: renamed from R17; footprint (none) -> Resistor_SMD:R_0603_1608Metric_Pad0.98x0.95mm_HandSolder
- renumbered J1 to J?, J3 to J?, J2 to J?, Q6 to Q?, Q7 to Q?, Q14 to Q?
Connections:
- net +BATT: now also BT?.1 (+), BT?.1 (+)
- net -BATT: now also R?.2, BT?.2 (-), BT?.2 (-), R102.1, R103.1, R104.1
- net LOAD-: now also C105.2
- net at Q?.1 (S), Q?.1 (S), Q?.2 (S)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: now also R?.2, C104.1, R102.2, R103.2, R104.2
- net at D?.2 (A): now also Q?.3 (D)
- new net: BT?.1 (+), BT?.2 (-) (x8)
- new net: C104.2, C105.1
Other:
- moved on the sheet: BT?, C?, D?, J?, NT?, Q?, R?
